File: Hardware/PCB.brd (EAGLE design)
At the start: 160 x 100 mm, 105 parts, among them IC1 BQ25180YBGR_BQ25180YBGR, IC2 DRV2605YZFR_DRV2605YZFR, IC3 BMA423_BMA423, IC9 RT6160AWSC_RT6160AWSC, J1 503480-2400_503480-2400, J2 KH-TYPE-C-16P_KH-TYPE-C-16P, J2\ TC2030-IDC_TC2030-IDC, Q1 20V/4.2A/52mΩ/1.4W, Q3 ESP32_C6_LIBRARY_6_SI1308EDL-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, U3 ESP32_C6_LIBRARY_MAX17048G+T10, X1 32MHz, X2 32.768kHz

Commit message: Design Validation (DVT)
Parts:
- removed C26, C28, C35, C36, C40, C41, C44, C45: 1uF, InkTime_v5:ESP32_C6_LIBRARY_1_ESP32_WROVER_EAGLE-LTSPICE_C0402
- removed C46: 4.7uF, InkTime_v5:ESP32_C6_LIBRARY_1_ESP32_WROVER_EAGLE-LTSPICE_C0402
- removed C47: 0.1uF, InkTime_v5:GRM011R60J152KE01L_2_CAPC0201X13N
- removed D1: ESP32_C6_LIBRARY_3_USBLC6-2SC6Y, InkTime_v5:ESP32_C6_LIBRARY_3_SOT95P280X145-6N
- removed J2: KH-TYPE-C-16P_KH-TYPE-C-16P, InkTime_v5:KH-TYPE-C-16P_KINGHELM_KH-TYPE-C-16P
- removed U$1: NORDIC_NRF_4_NRF52840_QF, InkTime_v5:NORDIC_NRF_4_AQFN50P700X700X85_HS-74N
- added D3: ESP32_C6_LIBRARY_3_USBLC6-2SC6Y, InkTime_v5:ESP32_C6_LIBRARY_3_SOT95P280X145-6N
- added EPD_C1, EPD_C10, EPD_C11, EPD_C12, EPD_C2, EPD_C7, EPD_C8, EPD_C9: 1uF/50V, InkTime_v5:ESP32_C6_LIBRARY_1_ESP32_WROVER_EAGLE-LTSPICE_C0402
- added EPD_C5: 0.1uF/50V, InkTime_v5:GRM011R60J152KE01L_2_CAPC0201X13N
- added EPD_C6: 1uF/5OV, InkTime_v5:ESP32_C6_LIBRARY_1_ESP32_WROVER_EAGLE-LTSPICE_C0402
- added J4: KH-TYPE-C-16P, InkTime_v5:KH-TYPE-C-16P_KINGHELM_KH-TYPE-C-16P
- added U1: NRF52840_QF, InkTime_v5:NORDIC_NRF_4_AQFN50P700X700X85_HS-74N
- ANT1: value 2450AT18B100E_2450AT18B100E -> 2450AT18B100E
- C42: value 1uF -> 0.1uF; device InkTime_v5:ESP32_C6_LIBRARY_1_ESP32_WROVER_EAGLE-LTSPICE_C0402 -> InkTime_v5:GRM011R60J152KE01L_2_CAPC0201X13N
- C43: value 0.1uF -> 4.7uF; device InkTime_v5:GRM011R60J152KE01L_2_CAPC0201X13N -> InkTime_v5:ESP32_C6_LIBRARY_1_ESP32_WROVER_EAGLE-LTSPICE_C0402
- D2, D4, D5: value ESP32_C6_LIBRARY_5_MBR0530 -> MBR0530
- IC3: value BMA423_BMA423 -> BMA423
- IC9: value RT6160AWSC_RT6160AWSC -> RT6160AWSC
- J2\: value TC2030-IDC_TC2030-IDC -> TC2030-IDC
- Q3: value ESP32_C6_LIBRARY_6_SI1308EDL-T1-GE3 -> SI1308EDL-T1-GE3
- R2, R3, R4: value CPF0201D7K68C1_CPF0201D7K68C1 -> 0
- moved D2 212.1 mm to (-1.75, -10.0), turned to 90 degrees
- moved TP_BAT_GND 205.5 mm to (18.9, 14.4)
- moved R7 205.4 mm to (6.48, -14.7)
- moved TP2 205.1 mm to (16.7, 15.0)
- moved L3 203.1 mm to (18.7, -0.60)
- moved R8 200.1 mm to (1.17, -10.2)
- moved L5 199.5 mm to (-5.23, -12.0)
- moved R_TYPE_SEL 199.5 mm to (-8.49, -8.17)
- moved C33 199.3 mm to (19.6, 10.9)
- moved TP1 199.0 mm to (14.0, 15.8)
- moved R_PWR_EPD 198.0 mm to (-1.06, -4.13)
- moved L1 198.0 mm to (14.5, -9.39)
- moved TP_SDA 197.3 mm to (21.1, 5.32)
- moved R18 196.5 mm to (20.5, 8.61)
- moved TP_3V3 196.5 mm to (-9.50, -4.15)
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Connections:
- net 3V3: now also IC9.E2, U1.P$A22, U1.P$AD14, U1.P$AD23, U1.P$B1, U1.P$W1, U1.P$Y2; no longer U$1.P$A22, U$1.P$AD14, U$1.P$AD23, U$1.P$B1, U$1.P$W1, U$1.P$Y2
- net ALERT: now also U1.P$J24; no longer U$1.P$J24
- net D+: now also D3.4, U1.P$AD6; no longer D1.4, U$1.P$AD6
- net D-: now also D3.6, U1.P$AD4; no longer D1.6, U$1.P$AD4
- net DEC1: now also U1.P$C1; no longer U$1.P$C1
- net DEC3: now also U1.P$D23; no longer U$1.P$D23
- net DEC4_6: now also U1.P$B5, U1.P$E24; no longer U$1.P$B5, U$1.P$E24
- net DN: now also D3.1, J4.A7, J4.B7; no longer D1.1, J2.A7, J2.B7
- net DP: now also D3.3, J4.A6, J4.B6; no longer D1.3, J2.A6, J2.B6
- net EPD_3V3: now also EPD_C5.1; no longer C43.1
- net EPD_BUSY: now also U1.P$AD12; no longer U$1.P$AD12
- net EPD_CS: now also U1.P$K2; no longer U$1.P$K2
- net EPD_DC: now also U1.P$AD10; no longer U$1.P$AD10
- net EPD_RST: now also U1.P$AC11; no longer U$1.P$AC11
- net GND: now also C42.2, D3.2, EPD_C1.1, EPD_C10.1, EPD_C11.1, EPD_C12.1, EPD_C2.1, EPD_C5.2, EPD_C6.1, EPD_C7.1, EPD_C8.1, EPD_C9.1, J4.A12_B1, J4.A1_B12, J4.SH1, J4.SH2, J4.SH3, J4.SH4, U1.P$74, U1.P$75, U1.P$76, U1.P$77, U1.P$78, U1.P$79, U1.P$80, U1.P$81, U1.P$82, U1.P$83, U1.P$84, U1.P$85, U1.P$86, U1.P$87, U1.P$88, U1.P$89, U1.P$90, U1.P$B7, U1.P$F23; no longer C26.1, C28.1, C35.1, C36.1, C40.1, C41.1, C42.1, C44.1, C45.1, C46.2, C47.2, D1.2, J2.A12_B1, J2.A1_B12, J2.SH1, J2.SH2, J2.SH3, J2.SH4, U$1.P$74, U$1.P$75, U$1.P$76, U$1.P$77, U$1.P$78, U$1.P$79, U$1.P$80, U$1.P$81, U$1.P$82, U$1.P$83, U$1.P$84, U$1.P$85, U$1.P$86, U$1.P$87, U$1.P$88, U$1.P$89, U$1.P$90, U$1.P$B7, U$1.P$F23
- net HAPTIC_EN: now also U1.P$U1; no longer U$1.P$U1
- net IMU_INT1: now also U1.P$N1; no longer U$1.P$N1
- net IMU_INT2: now also U1.P$P2; no longer U$1.P$P2
- net LX1: no longer IC9.B3
- net MOSI: now also U1.P$B13; no longer U$1.P$B13
- net N$1: now also J4.A5; no longer J2.A5
- net N$11: now also U1.P$A18; no longer U$1.P$A18
- net N$12: now also U1.P$H23; no longer U$1.P$H23
- net N$13: now also U1.P$AC5; no longer U$1.P$AC5
- net N$16: now also U1.P$N24; no longer U$1.P$N24
- net N$20: now also EPD_C2.2; no longer C42.2
- net N$21: now also EPD_C1.2; no longer C41.2
- net N$23: now also J4.B5; no longer J2.B5
- net N$29: now also EPD_C12.2; no longer C26.2
- net N$31: now also EPD_C10.2; no longer C29.2
- net N$33: now also EPD_C8.2; no longer C31.2
- net N$34: now also EPD_C7.2; no longer C35.2
- net N$35: now also EPD_C6.2; no longer C36.2
- net N$5: now also U1.P$A23; no longer U$1.P$A23
- net N$7: now also U1.P$B3; no longer U$1.P$B3
- net N$9: now also U1.P$B24; no longer U$1.P$B24
- net P0.00: now also U1.P$D2; no longer U$1.P$D2
- net P0.01: now also U1.P$F2; no longer U$1.P$F2
- net P0.04: now also U1.P$J1; no longer U$1.P$J1
- net P0.09: now also U1.P$L24; no longer U$1.P$L24
- net P0.13: now also C30.2, U1.P$AD8; no longer C40.2, U$1.P$AD8
- net P0.14: now also C31.2, U1.P$AC9; no longer C44.2, U$1.P$AC9
- net P0.19: now also U1.P$AC15; no longer U$1.P$AC15
- net P0.20: now also U1.P$AD16; no longer U$1.P$AD16
- net P0.21: now also U1.P$AC17; no longer U$1.P$AC17
- net P0.22: now also U1.P$AD18; no longer U$1.P$AD18
- net P0.23: now also U1.P$AC19; no longer U$1.P$AC19
- net P0.24: now also U1.P$AD20; no longer U$1.P$AD20
- net P0.25: now also U1.P$AC21; no longer U$1.P$AC21
- net P0.26: now also U1.P$G1; no longer U$1.P$G1
- net P0.27: now also U1.P$H2; no longer U$1.P$H2
- net P0.28: now also U1.P$B11; no longer U$1.P$B11
- net P0.29: now also U1.P$A10; no longer U$1.P$A10
- net P0.30: now also U1.P$B9; no longer U$1.P$B9
- net P0.31: now also U1.P$A8; no longer U$1.P$A8
- net P1.01: now also U1.P$Y23; no longer U$1.P$Y23
- net P1.02: now also C29.2, U1.P$W24; no longer C45.2, U$1.P$W24
- net P1.03: now also U1.P$V23; no longer U$1.P$V23
- net P1.04: now also U1.P$U24; no longer U$1.P$U24
- net P1.05: now also U1.P$T23; no longer U$1.P$T23
- net P1.06: now also U1.P$R24; no longer U$1.P$R24
- net P1.07: now also U1.P$P23; no longer U$1.P$P23
- net P1.09: now also U1.P$R1; no longer U$1.P$R1
- net P1.10: now also U1.P$A20; no longer U$1.P$A20
- net P1.11: now also U1.P$B19; no longer U$1.P$B19
- net P1.12: now also U1.P$B17; no longer U$1.P$B17
- net P1.13: now also U1.P$A16; no longer U$1.P$A16
- net P1.14: now also U1.P$B15; no longer U$1.P$B15
- net P1.15: now also U1.P$A14; no longer U$1.P$A14
- net PMIC_INT: now also U1.P$T2; no longer U$1.P$T2
- net PREVGH: now also EPD_C9.2; no longer C30.2
- net PREVGL: now also EPD_C11.2; no longer C28.2
- net RESET: now also U1.P$AC13; no longer U$1.P$AC13
- net SCK: now also U1.P$A12; no longer U$1.P$A12
- net SCL: now also U1.P$M2; no longer U$1.P$M2
- net SDA: now also U1.P$L1; no longer U$1.P$L1
- net SWDCLK: now also U1.P$AA24; no longer U$1.P$AA24
- net SWDIO: now also U1.P$AC24; no longer U$1.P$AC24
- net SWO: now also U1.P$AD22; no longer U$1.P$AD22
- net VBUS: now also C42.1, C43.1, D3.5, J4.A4_B9, J4.A9_B4, U1.P$AD2; no longer C46.1, C47.1, D1.5, J2.A4_B9, J2.A9_B4, U$1.P$AD2
Routing:
- net GND: track 0.00 -> 375.1 mm, vias 0 -> 6
- net 3V3: track 0.00 -> 144.2 mm, vias 0 -> 14
- net SDA: track 0.00 -> 76.4 mm, vias 0 -> 6
- net SCL: track 0.00 -> 59.3 mm, vias 0 -> 9
- net VBUS: track 0.00 -> 47.9 mm, vias 0 -> 4
- net P0.13: track 0.00 -> 47.6 mm, vias 0 -> 4
- net SCK: track 0.00 -> 46.1 mm, vias 0 -> 2
- net N$12: track 0.00 -> 41.8 mm, vias 0 -> 4
- net VREG: track 0.00 -> 35.4 mm, vias 0 -> 6
- net N$18: track 0.00 -> 30.4 mm, vias 0 -> 3
- net MOSI: track 0.00 -> 29.1 mm, vias 0 -> 8
- net DEC4_6: track 0.00 -> 29.0 mm, vias 0 -> 5
- net SWDCLK: track 0.00 -> 28.4 mm, vias 0 -> 4
- net P0.14: track 0.00 -> 27.9 mm, vias 0 -> 2
- net RESET: track 0.00 -> 26.8 mm, vias 0 -> 9
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- added copper zone on layer 1, net GND
- added copper zone on layer 16, net GND
Other:
- board size 160 x 100 mm -> 46 x 35 mm
