File: Hardware/Schematic.sch (EAGLE design)
At the start: 105 parts, among them IC1 BQ25180YBGR_BQ25180YBGR, IC2 DRV2605YZFR_DRV2605YZFR, IC3 BMA423_BMA423, IC9 RT6160AWSC_RT6160AWSC, J1 503480-2400_503480-2400, J2 KH-TYPE-C-16P_KH-TYPE-C-16P, J2\ TC2030-IDC_TC2030-IDC, Q1 20V/4.2A/52mΩ/1.4W, Q3 ESP32_C6_LIBRARY_6_SI1308EDL-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, U3 ESP32_C6_LIBRARY_MAX17048G+T10, X1 32MHz, X2 32.768kHz

Commit message: Design Validation (DVT)
Parts:
- removed C40, C44, C45: 1uF, InkTime_v5:ESP32_C6_LIBRARY_1_ESP32_WROVER_EAGLE-LTSPICE_CC0402
- removed C46: 4.7uF, InkTime_v5:ESP32_C6_LIBRARY_1_ESP32_WROVER_EAGLE-LTSPICE_CC0402
- removed C47: 0.1uF, InkTime_v5:GRM011R60J152KE01L_2_GRM011R60J152KE01L
- added EPD_C10, EPD_C2, EPD_C8, EPD_C9: 1uF/50V, InkTime_v5:ESP32_C6_LIBRARY_1_ESP32_WROVER_EAGLE-LTSPICE_CC0402
- added EPD_C5: 0.1uF/50V, InkTime_v5:GRM011R60J152KE01L_2_GRM011R60J152KE01L
- ANT1: value 2450AT18B100E_2450AT18B100E -> 2450AT18B100E; SPICEPREFIX (none) -> B
- C42: value 1uF -> 0.1uF; device InkTime_v5:ESP32_C6_LIBRARY_1_ESP32_WROVER_EAGLE-LTSPICE_CC0402 -> InkTime_v5:GRM011R60J152KE01L_2_GRM011R60J152KE01L
- C43: value 0.1uF -> 4.7uF; device InkTime_v5:GRM011R60J152KE01L_2_GRM011R60J152KE01L -> InkTime_v5:ESP32_C6_LIBRARY_1_ESP32_WROVER_EAGLE-LTSPICE_CC0402
- D2, D4, D5: value ESP32_C6_LIBRARY_5_MBR0530 -> MBR0530
- EPD_C1, EPD_C11, EPD_C12, EPD_C7: value 1uF -> 1uF/50V
- EPD_C6: value 1uF -> 1uF/5OV
- IC3: value BMA423_BMA423 -> BMA423
- IC9: value RT6160AWSC_RT6160AWSC -> RT6160AWSC
- J2\: value TC2030-IDC_TC2030-IDC -> TC2030-IDC
- J4: value KH-TYPE-C-16P_KH-TYPE-C-16P -> KH-TYPE-C-16P
- Q3: value ESP32_C6_LIBRARY_6_SI1308EDL-T1-GE3 -> SI1308EDL-T1-GE3
- R2, R3, R4: value CPF0201D7K68C1_CPF0201D7K68C1 -> 0
- U1: value NORDIC_NRF_4_NRF52840_QF -> NRF52840_QF
- renumbered C26 to EPD_C12, C28 to EPD_C11, C35 to EPD_C7, C36 to EPD_C6, C41 to EPD_C1, D1 to D3, J2 to J4, U$1 to U1
Connections:
- net 3V3: now also IC9.VOUT_1
- net EPD_3V3: now also EPD_C5.1; no longer C43.1
- net GND: now also C42.2, EPD_C10.1, EPD_C2.1, EPD_C5.2, EPD_C8.1, EPD_C9.1; no longer C40.1, C42.1, C44.1, C45.1, C46.2, C47.2
- net LX1: no longer IC9.SW1_2
- net N$20: now also EPD_C2.2; no longer C42.2
- net N$31: now also EPD_C10.2; no longer C29.2
- net N$33: now also EPD_C8.2; no longer C31.2
- net P0.13: now also C30.2; no longer C40.2
- net P0.14: now also C31.2; no longer C44.2
- net P1.02: now also C29.2; no longer C45.2
- net PREVGH: now also EPD_C9.2; no longer C30.2
- net VBUS: now also C42.1, C43.1; no longer C46.1, C47.1
Other:
- moved on the sheet: C20, C23, C24, C25, C29, C30, C31, C33, C42, C43, C7, R2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
